File: CleverCoffe_ESP32_PidOnly_Plus/CleverCoffe_ESP32_PidOnly_Plus.kicad_pcb (KiCad board)
At the start: 2 copper layers, 75 x 50 mm, 17 parts

Commit message: User 3-pole solder jumpers for voltage selection
Parts:
- removed JP1, JP2, JP3, JP4: SolderJumper_2_Open, Jumper:SolderJumper-2_P1.3mm_Open_Pad1.0x1.5mm
- added VS1: Voltage Jumper, Jumper:SolderJumper-3_P1.3mm_Open_Pad1.0x1.5mm_NumberLabels, B.Cu at (151.8, 109.5)
- added VS2: Voltage Jumper, Jumper:SolderJumper-3_P1.3mm_Open_Pad1.0x1.5mm_NumberLabels, B.Cu at (127.2, 109.5)
- moved ESP1 0.25 mm to (104.8, 104.0)
