File: wiring_diagrams/ESP32_minimal_full_featured_Silvia_E.kicad_sch (KiCad schematic)
At the start: 23 parts

Commit message: Fix error in wiring diagram for Silvia E
Parts:
- added CPU: ~, symbol User:Silvia_E_CPU
- added D3: 12V LED, symbol Device:LED
Connections:
- net at Power_Supply.1 (L), Thermal_Safety.1 (A), Water_Switch.1: now also AC_Mains.3 (L), CPU.2; no longer Power_Switch.4
- net at 3WV_SSR.11, 3_Way_Valve.2 (N), Heater_SSR.11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: now also CPU.10; no longer Power_Switch.3
- net at Pump_SSR.14, Vibration_Pump.1 (L), Water_Switch.4: now also CPU.3
- net at Power_Switch.1: now also CPU.6; no longer AC_Mains.3 (L)
- net at AC_Mains.2 (N): now also CPU.1, CPU.9; no longer Power_Switch.2
- new net: CPU.5, D3.1 (K), Power_Switch.4
- new net: CPU.7, D3.2 (A)
Other:
- title: ESP32 Minimal PCB - Full Featured Build -> ESP32 Minimal PCB - Full Featured Build for Silvia E
- moved on the sheet: AC_Mains, Brew_Switch, D1, D2, Power_Switch, R1, R2, Steam_Switch, Water_Switch
