File: CleverCoffee_ESP32_Dev_SMD/CleverCoffee_ESP32_Dev_SMD.kicad_sch (KiCad schematic)
At the start: 28 parts

Commit message: Add new SMD variant of the Dev PCB, make naming scheme consistent
Parts:
- removed BS_LED1: Conn_01x02, Connector_PinSocket_2.54mm:PinSocket_1x03_P2.54mm_Vertical, symbol Connector_Generic:Conn_01x03
- removed C3: 100 nF, Capacitor_THT:C_Axial_L5.1mm_D3.1mm_P7.50mm_Horizontal, symbol Device:C
- C1: footprint Capacitor_THT:CP_Radial_D8.0mm_P3.80mm -> Capacitor_SMD:CP_Elec_6.3x7.7
- C2: footprint Capacitor_THT:C_Axial_L5.1mm_D3.1mm_P7.50mm_Horizontal -> Capacitor_SMD:C_1206_3216Metric_Pad1.33x1.80mm_HandSolder
- R1, R2, R3, R6, R7, R8, R9: footprint Resistor_THT:R_Axial_DIN0207_L6.3mm_D2.5mm_P10.16mm_Horizontal -> Resistor_SMD:R_1206_3216Metric_Pad1.30x1.75mm_HandSolder
- R4: renamed from R5; footprint Resistor_THT:R_Axial_DIN0207_L6.3mm_D2.5mm_P10.16mm_Horizontal -> Resistor_SMD:R_1206_3216Metric_Pad1.30x1.75mm_HandSolder
- R5: renamed from R4; footprint Resistor_THT:R_Axial_DIN0207_L6.3mm_D2.5mm_P10.16mm_Horizontal -> Resistor_SMD:R_1206_3216Metric_Pad1.30x1.75mm_HandSolder
- SBS_LED1: renamed from S_LED1; value Conn_01x03 -> Conn_01x05; footprint Connector_PinSocket_2.54mm:PinSocket_1x03_P2.54mm_Vertical -> Connector_PinSocket_2.54mm:PinSocket_1x05_P2.54mm_Vertical; symbol Connector_Generic:Conn_01x03 -> Connector_Generic:Conn_01x05
Connections:
- net +5V: now also SBS_LED1.4 (Pin_4); no longer SBS_LED1.2 (Pin_2)
- net GND: now also SBS_LED1.5 (Pin_5); no longer SBS_LED1.3 (Pin_3)
- net at R5.1: now also SBS_LED1.2 (Pin_2)
- net at R6.1: now also SBS_LED1.3 (Pin_3)
Other:
- note added: "Status LED Brew LED Steam LED"
- note removed: "Brew LED Steam LED"
- note removed: "Status LED"
- moved on the sheet: JP1, R4, R5, R6
