File: CleverCoffee_ESP32_Dev_SMD/CleverCoffee_ESP32_Dev_SMD.kicad_pcb (KiCad board)
At the start: 2 copper layers, 85 x 60 mm, 32 parts

Commit message: Updated Gerber files for all PCBs
Parts:
- renumbered I2C1 to I2C
Routing:
- net SDA: track 63.6 -> 60.7 mm
- net IO1: track 48.6 -> 48.1 mm
Other:
- board text added: "CleverCoffee ESP32 Dev SMD Rev 1.0 23a4cb6"
- board text removed: "CleverCoffee ESP32 Dev SMD Rev 1.0 29ba717"
