File: CleverCoffee_ESP32_Dev/CleverCoffee_ESP32_Dev.kicad_pcb (KiCad board)
At the start: 2 copper layers, 95 x 65 mm, 35 parts

Commit message: Add new SMD variant of the Dev PCB, make naming scheme consistent
Parts:
- removed C3: 100 nF, Capacitor_THT:C_Axial_L5.1mm_D3.1mm_P7.50mm_Horizontal

Commit message: Updated Gerber files for all PCBs
Other:
- board text added: "CleverCoffee ESP32 Dev Rev 1.6 23a4cb6"
- board text removed: "29ba717"
- board text removed: "CleverCoffee ESP32 Rev 1.6"
Changed lines of the file:
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@@
     (effects (font (size 0.5 0.5) (thickness 0.1)))
-  )
-  (gr_text "29ba717" (at 146.56 116.78) (layer "F.SilkS")
-    (effects (font (size 0.85 0.85) (thickness 0.15) bold) (justify left bottom))
   )
   (gr_text "3.3V" (at 187.275 121.95 90) (layer "F.SilkS")
@@
     (effects (font (size 0.5 0.5) (thickness 0.1)))
   )
-  (gr_text "CleverCoffee ESP32 Rev 1.6\n" (at 141.48 114.37) (layer "F.SilkS")
+  (gr_text "CleverCoffee ESP32 Dev\nRev 1.6 23a4cb6\n" (at 141.48 114.37) (layer "F.SilkS")
     (effects (font (size 1 1) (thickness 0.15)))
   )
