File: ABP2_Breakoutboard/KiCad/APB2_Breakout.kicad_pcb (KiCad board)
At the start: 2 copper layers, 35.6 x 26.9 mm, 7 parts, among them J1 Screw_Terminal_01x04, J2 Screw_Terminal_01x04

Commit message: move pin names on silk, add logo and PCB name
Parts:
- added REF**: OSHW-Logo2_7.3x6mm_SilkScreen, Symbol:OSHW-Logo2_7.3x6mm_SilkScreen, F.Cu at (158.0, 119.5)
Routing:
- net 3V3: track 42.7 -> 43.5 mm
Other:
- board text added: "CleverCoffee ABP2 i2c Rev 1.1"
